File: ESP32-Geiger-Counter.kicad_sch (KiCad schematic)
At the start: 82 parts, among them J1 2s1p Lipo Battery Pack (8.4V-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, J2 USB_C_Receptacle_USB2.0_16P, J3 SBM20 +, J4 SBM20 -, J5 Conn_01x07, Q1 Q_NMOS_GDS, Q2 2N3904, Q3 2N7002, Q4 AO3401A, SW1 SW_SPDT, SW2 RESET, SW3 BOOT, U1 BQ25886RGE, U2 AP63203WU, U3 ESP32-S3-WROOM-1, U4 UCC27517DBVR, U5 USBLC6-2SC6

Commit message: misc
Parts:
- J1: footprint (none) -> Connector_JST:JST_XH_S2B-XH-A_1x02_P2.50mm_Horizontal
- L2: footprint (none) -> Inductor_SMD:L_Bourns-SRN6028
Other:
- note added: "(Between 8.4-6V)"
- note added: "3.3V Buck Converter - P"
- note added: "https://www.digikey.com/en/products/detail/bourns-inc/SRN6028C-3R9M/17126460"
- note removed: "3.3V Buck Converter"
Changed lines of the file:
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@@
 		)
 	)
+	(text "(Between 8.4-6V)"
+		(exclude_from_sim no)
+		(at 243.84 113.03 0)
+		(effects
+			(font
+				(size 1.27 1.27)
+			)
+		)
+	)
 	(text "Piezo"
 		(exclude_from_sim no)
@@
 		)
 	)
+	(text "https://www.digikey.com/en/products/detail/bourns-inc/SRN6028C-3R9M/17126460"
+		(exclude_from_sim no)
+		(at 295.91 104.14 0)
+		(effects
+			(font
+				(size 1.27 1.27)
+			)
+		)
+	)
 	(text "Battery Connector "
 		(exclude_from_sim no)
@@
 		)
 	)
-	(text "3.3V Buck Converter"
+	(text "3.3V Buck Converter - P"
 		(exclude_from_sim no)
 		(at 251.206 93.98 0)
@@
 			)
 		)
-		(property "Footprint" ""
+		(property "Footprint" "Connector_JST:JST_XH_S2B-XH-A_1x02_P2.50mm_Horizontal"
 			(at 64.77 46.99 0)
 			(hide yes)
@@
 			)
 		)
-		(property "Footprint" ""
+		(property "Footprint" "Inductor_SMD:L_Bourns-SRN6028"
 			(at 298.45 111.76 0)
 			(hide yes)

Commit message: footprints
Parts:
- L1: footprint (none) -> SRP4020TA-1R0M:IND_SRP4020TA-1R0M
Other:
- moved on the sheet: R8, R9
Changed lines of the file:
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@@
 	(wire
 		(pts
+			(xy 180.34 87.63) (xy 180.34 86.36)
+		)
+		(stroke
+			(width 0)
+			(type default)
+		)
+	)
+	(wire
+		(pts
 			(xy 435.61 234.95) (xy 445.77 234.95)
 		)
@@
 	(wire
 		(pts
+			(xy 173.99 87.63) (xy 173.99 86.36)
+		)
+		(stroke
+			(width 0)
+			(type default)
+		)
+	)
+	(wire
+		(pts
 			(xy 251.46 130.81) (xy 251.46 133.35)
 		)
@@
 	(wire
 		(pts
-			(xy 180.34 104.14) (xy 180.34 93.98)
+			(xy 180.34 104.14) (xy 180.34 95.25)
 		)
 		(stroke
@@
 	(wire
 		(pts
-			(xy 173.99 101.6) (xy 173.99 93.98)
+			(xy 173.99 101.6) (xy 173.99 95.25)
 		)
 		(stroke
@@
 	(symbol
 		(lib_id "Device:R_US")
-		(at 180.34 90.17 180)
+		(at 180.34 91.44 180)
 		(unit 1)
 		(body_style 1)
@@
 		(dnp no)
 		(property "Reference" "R9"
-			(at 184.15 89.662 0)
+			(at 184.15 90.932 0)
 			(show_name no)
 			(do_not_autoplace no)
@@
 		)
 		(property "Value" "2.2K"
-			(at 184.658 91.694 0)
+			(at 184.658 92.964 0)
 			(show_name no)
 			(do_not_autoplace no)
@@
 		)
 		(property "Footprint" "Resistor_SMD:R_0805_2012Metric"
-			(at 179.324 89.916 90)
+			(at 179.324 91.186 90)
 			(hide yes)
 			(show_name no)
@@
 		)
 		(property "Datasheet" ""
-			(at 180.34 90.17 0)
+			(at 180.34 91.44 0)
 			(hide yes)
 			(show_name no)
@@
 		)
 		(property "Description" "Resistor, US symbol"
-			(at 180.34 90.17 0)
+			(at 180.34 91.44 0)
 			(hide yes)
 			(show_name no)
@@
 			)
 		)
-		(property "Footprint" ""
+		(property "Footprint" "SRP4020TA-1R0M:IND_SRP4020TA-1R0M"
 			(at 195.58 111.76 0)
 			(hide yes)
@@
 	(symbol
 		(lib_id "Device:R_US")
-		(at 173.99 90.17 180)
+		(at 173.99 91.44 180)
 		(unit 1)
 		(body_style 1)
@@
 		(dnp no)
 		(property "Reference" "R8"
-			(at 171.45 88.646 0)
+			(at 171.45 89.916 0)
 			(show_name no)
 			(do_not_autoplace no)
@@
 		)
 		(property "Value" "2.2K"
-			(at 170.18 90.678 0)
+			(at 170.18 91.948 0)
 			(show_name no)
 			(do_not_autoplace no)
@@
 		)
 		(property "Footprint" "Resistor_SMD:R_0805_2012Metric"
-			(at 172.974 89.916 90)
+			(at 172.974 91.186 90)
 			(hide yes)
 			(show_name no)
@@
 		)
 		(property "Datasheet" ""
-			(at 173.99 90.17 0)
+			(at 173.99 91.44 0)
 			(hide yes)
 			(show_name no)
@@
 		)
 		(property "Description" "Resistor, US symbol"
-			(at 173.99 90.17 0)
+			(at 173.99 91.44 0)
 			(hide yes)
 			(show_name no)

Commit message: general updates
Parts:
- BZ1: footprint (none) -> CPT_2207_95_SMT_TR:XDCR_CPT-2207-95-SMT-TR
- J5: footprint (none) -> Connector_PinSocket_2.54mm:PinSocket_1x07_P2.54mm_Vertical
- Q1: value Q_NMOS_GDS -> STN1HNK60
- Q2: footprint Package_TO_SOT_THT:TO-92_Inline -> Package_TO_SOT_SMD:SOT-23
Other:
- moved on the sheet: C19, C20, C21, C22, C23, C24, C25, C26, C27, C28, C29, D3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

Commit message: replaced piezo
Parts:
- BZ1: footprint CPT_2207_95_SMT_TR:XDCR_CPT-2207-95-SMT-TR -> CPT_1203_78_SMT_TR:XDCR_CPT-1203-78-SMT-TR
Changed lines of the file:
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@@
 			)
 		)
-		(property "Footprint" "CPT_2207_95_SMT_TR:XDCR_CPT-2207-95-SMT-TR"
+		(property "Footprint" "CPT_1203_78_SMT_TR:XDCR_CPT-1203-78-SMT-TR"
 			(at 283.845 40.64 90)
 			(hide yes)

Commit message: added sbm20 footprint
Parts:
- removed J3: SBM20 +, symbol Connector_Generic:Conn_01x01
- removed J4: SBM20 -, symbol Connector_Generic:Conn_01x01
- added U6: SBM-20 Geiger Mueller Tube, symbol Custom Parts:Geiger_Mueller_Tube
Connections:
- net at R20.2, R21.1: now also U6.2 (K)
- net at R19.2: now also U6.1 (A)
Changed lines of the file:
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@@
 		)
 	)
-	(rectangle
-		(start 396.24 200.66)
-		(end 425.45 210.82)
-		(stroke
-			(width 0)
-			(type default)
-		)
-		(fill
-			(type none)
-		)
-	)
 	(text "2s1p Battery Charging"
 		(exclude_from_sim no)
@@
 	(wire
 		(pts
+			(xy 420.37 204.47) (xy 434.34 204.47)
+		)
+		(stroke
+			(width 0)
+			(type default)
+		)
+	)
+	(wire
+		(pts
 			(xy 180.34 87.63) (xy 180.34 86.36)
 		)
@@
 	(wire
 		(pts
-			(xy 397.51 204.47) (xy 389.89 204.47)
+			(xy 389.89 204.47) (xy 401.32 204.47)
 		)
 		(stroke
@@
 	(wire
 		(pts
-			(xy 422.91 204.47) (xy 434.34 204.47)
-		)
-		(stroke
-			(width 0)
-			(type default)
-		)
-	)
-	(wire
-		(pts
 			(xy 76.2 101.6) (xy 76.2 105.41)
 		)
@@
 	)
 	(symbol
-		(lib_id "Connector_Generic:Conn_01x01")
-		(at 417.83 204.47 180)
-		(unit 1)
-		(body_style 1)
-		(exclude_from_sim no)
-		(in_bom yes)
-		(on_board yes)
-		(in_pos_files yes)
-		(dnp no)
-		(property "Reference" "J4"
-			(at 414.02 204.47 0)
-			(show_name no)
-			(do_not_autoplace no)
-			(effects
-				(font
-					(size 1.27 1.27)
-				)
-			)
-		)
-		(property "Value" "SBM20 -"
-			(at 419.1 208.28 0)
-			(show_name no)
-			(do_not_autoplace no)
-			(effects
-				(font
-					(size 1.27 1.27)
-				)
-			)
-		)
-		(property "Footprint" ""
-			(at 417.83 204.47 0)
-			(hide yes)
-			(show_name no)
-			(do_not_autoplace no)
-			(effects
-				(font
-					(size 1.27 1.27)
-				)
-			)
-		)
-		(property "Datasheet" ""
-			(at 417.83 204.47 0)
-			(hide yes)
-			(show_name no)
-			(do_not_autoplace no)
-			(effects
-				(font
-					(size 1.27 1.27)
-				)
-			)
-		)
-		(property "Description" "Generic connector, single row, 01x01, script generated (kicad-library-utils/schlib/autogen/connector/)"
-			(at 417.83 204.47 0)
-			(hide yes)
-			(show_name no)
-			(do_not_autoplace no)
-			(effects
-				(font
-					(size 1.27 1.27)
-				)
-			)
-		)
-		(pin "1"
-		)
-		(instances
-			(project "ESP32-Geiger-Counter"
-				(path "/1d04c1b6-b1c1-45fc-a2be-06365cafa415"
-					(reference "J4")
-					(unit 1)
-				)
-			)
-		)
-	)
-	(symbol
 		(lib_id "power:GND")
 		(at 78.74 208.28 180)
@@
 	)
 	(symbol
+		(lib_id "Custom Parts:Geiger_Mueller_Tube")
+		(at 407.67 208.28 90)
+		(unit 1)
+		(body_style 1)
+		(exclude_from_sim no)
+		(in_bom yes)
+		(on_board yes)
+		(in_pos_files yes)
+		(dnp no)
+		(property "Reference" "U6"
+			(at 411.0953 196.534 90)
+			(show_name no)
+			(do_not_autoplace no)
+			(effects
+				(font
+					(size 1.27 1.27)
+				)
+			)
+		)
+		(property "Value" "SBM-20 Geiger Mueller Tube"
+			(at 411.4353 198.8233 90)
+			(show_name no)
+			(do_not_autoplace no)
+			(effects
+				(font
+					(size 1.27 1.27)
+				)
+			)
+		)
+		(property "Footprint" ""
+			(at 407.67 208.28 0)
+			(hide yes)
+			(show_name no)
+			(do_not_autoplace no)
+			(effects
+				(font
+					(size 1.27 1.27)
+				)
+			)
+		)
+		(property "Datasheet" ""
+			(at 407.67 208.28 0)
+			(hide yes)
+			(show_name no)
+			(do_not_autoplace no)
+			(effects
+				(font
+					(size 1.27 1.27)
+				)
+			)
+		)
+		(property "Description" ""
+			(at 407.67 208.28 0)
+			(hide yes)
+			(show_name no)
+			(do_not_autoplace no)
+			(effects
+				(font
+					(size 1.27 1.27)
+				)
+			)
+		)
+		(pin "1"
+		)
+		(pin "2"
+		)
+		(instances
+			(project "ESP32-Geiger-Counter"
+				(path "/1d04c1b6-b1c1-45fc-a2be-06365cafa415"
+					(reference "U6")
+					(unit 1)
+				)
+			)
+		)
+	)
+	(symbol
 		(lib_id "power:GND")
 		(at 279.4 77.47 0)
@@
 					(unit 1)
 				)
-			)
-		)
-	)
-	(symbol
-		(lib_id "Connector_Generic:Conn_01x01")
-		(at 402.59 204.47 0)
-		(unit 1)
-		(body_style 1)
-		(exclude_from_sim no)
-		(in_bom yes)
-		(on_board yes)
-		(in_pos_files yes)
-		(dnp no)
-		(property "Reference" "J3"
-			(at 405.13 203.1999 0)
-			(show_name no)
-			(do_not_autoplace no)
-			(effects
-				(font
-					(size 1.27 1.27)
-				)
-				(justify left)
-			)
-		)
-		(property "Value" "SBM20 +"
-			(at 400.05 208.28 0)
-			(show_name no)
-			(do_not_autoplace no)
-			(effects
-				(font
-					(size 1.27 1.27)
-				)
-				(justify left)
-			)
-		)
-		(property "Footprint" ""
-			(at 402.59 204.47 0)
-			(hide yes)
-			(show_name no)
-			(do_not_autoplace no)
-			(effects
-				(font
-					(size 1.27 1.27)
-				)
-			)
-		)
-		(property "Datasheet" ""
-			(at 402.59 204.47 0)
-			(hide yes)
-			(show_name no)
-			(do_not_autoplace no)
-			(effects
-				(font
-					(size 1.27 1.27)
-				)
-			)
-		)
-		(property "Description" "Generic connector, single row, 01x01, script generated (kicad-library-utils/schlib/autogen/connector/)"
-			(at 402.59 204.47 0)
-			(hide yes)
-			(show_name no)
-			(do_not_autoplace no)
-			(effects
-				(font
-					(size 1.27 1.27)
-				)
-			)
-		)
-		(pin "1"
-		)
-		(instances
-			(project "ESP32-Geiger-Counter"
-				(path "/1d04c1b6-b1c1-45fc-a2be-06365cafa415"
-					(reference "J3")
-					(unit 1)
-				)

Commit message: general stuff
Parts:
- removed Q2: 2N3904, Package_TO_SOT_SMD:SOT-23, symbol Transistor_BJT:2N3904
- added H1, H2, H3, H4: MountingHole, MountingHole:MountingHole_3.2mm_M3, symbol Mechanical:MountingHole
- added Q5: MMBT3904, Package_TO_SOT_SMD:SOT-23, symbol Transistor_BJT:MMBT3904
- R18: footprint Resistor_SMD:R_0805_2012Metric -> Resistor_SMD:R_1206_3216Metric
- U4: footprint footprints:DBV5_TEX -> UCC27517:DBV5_TEX
- U6: footprint (none) -> 3529:SBM-20 Tube
Connections:
- net GND: now also Q5.2 (E)
- net PULSE: now also Q5.3 (C)
- net at R21.2: now also Q5.1 (B)

Commit message: working on layout
Parts:
- C17: footprint Capacitor_SMD:C_0805_2012Metric -> Capacitor_SMD:C_1206_3216Metric
- J5: footprint Connector_PinSocket_2.54mm:PinSocket_1x07_P2.54mm_Vertical -> footprints:OLED_2.42in_SSD1309_SPI_7pin
Changed lines of the file:
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@@
 			)
 		)
-		(property "Footprint" "Capacitor_SMD:C_0805_2012Metric"
+		(property "Footprint" "Capacitor_SMD:C_1206_3216Metric"
 			(at 317.5 115.57 0)
 			(hide yes)
@@
 			)
 		)
-		(property "Footprint" "Connector_PinSocket_2.54mm:PinSocket_1x07_P2.54mm_Vertical"
+		(property "Footprint" "footprints:OLED_2.42in_SSD1309_SPI_7pin"
 			(at 344.17 40.64 0)
 			(hide yes)

Commit message: board layout changes
Parts:
- SW2, SW3: footprint Button_Switch_SMD:SW_SPST_TL3342 -> Button_Switch_THT:SW_PUSH_6mm
Changed lines of the file:
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@@
 			)
 		)
-		(property "Footprint" "Button_Switch_SMD:SW_SPST_TL3342"
+		(property "Footprint" "Button_Switch_THT:SW_PUSH_6mm"
 			(at 60.96 228.6 0)
 			(hide yes)
@@
 			)
 		)
-		(property "Footprint" "Button_Switch_SMD:SW_SPST_TL3342"
+		(property "Footprint" "Button_Switch_THT:SW_PUSH_6mm"
 			(at 60.96 213.36 0)
 			(hide yes)
